File: hardware/pcb/pax-button.kicad_pcb (KiCad board)
At the start: 2 copper layers, 70 x 70 mm, 13 parts, among them J1 BATTERY 4xAA NiMH, J2 LED RING, J3 GND x3, SW1 MX switch, U1 ESP32-C3 SuperMini

Commit message: Board v0.2, button auto-sleep, low-battery warning, shell guidance
Board: optional battery-gauge divider (R2/R3) to an ADC pin, C1 moved
outward to clear 50 mm rings, a write-on number box on the back. DRC
clean; new manufacturing zip. Firmware: deep-sleeps after ten minutes
without hearing the hub, wakes on a press. App: low-battery chip naming
the player. Build guide: guided dome, hard stop, board support, ring
shelf and antenna clearance for whoever models the shell.

Co-Authored-By: Claude Fable 5.1 <noreply@anthropic.com>
Parts:
- added R2: 100k (optional), R_Axial_DIN0207_L6.3mm_D2.5mm_P5.08mm_Vertical, F.Cu at (120.5, 92.0)
- added R3: 100k (optional), R_Axial_DIN0207_L6.3mm_D2.5mm_P5.08mm_Vertical, F.Cu at (124.0, 92.0)
- moved C1 6.21 mm to (124.8, 112.0)
Connections:
- net IO_A renamed VSENSE
Routing:
- net VBAT: track 9.50 -> 75.0 mm
- net VSENSE: track 2.54 -> 27.5 mm
- net +5V: track 77.8 -> 82.5 mm
Other:
- board text added: "No."
- board text added: "R2 R3 100k:"
- board text added: "battery gauge"
- board text added: "button v0.2"
- board text removed: "button v0.1"
